File: ADCModule.kicad_sch (KiCad schematic)
At the start: 15 parts, among them U1 OPA4197xD, U2 Opamp_Quad, U3 MCP3008

Commit message: Pushing updated schematics
Parts:
- removed U1: OPA4197xD, Package_SO:SOIC-14_3.9x8.7mm_P1.27mm, symbol Amplifier_Operational:OPA4197xD
- removed U2: Opamp_Quad, symbol Device:Opamp_Quad
- added J10, J4, J5, J9: Conn_01x03_Pin, symbol Connector:Conn_01x03_Pin
- added U13, U15: OPA4197xD, Package_SO:SOIC-14_3.9x8.7mm_P1.27mm, symbol Amplifier_Operational:OPA4197xD
- renumbered U3 to U2
Connections:
- net +15V: now also U13.4 (V+), U15.4 (V+)
- net +5V: now also J10.2 (Pin_2), J4.2 (Pin_2), J5.2 (Pin_2), J9.2 (Pin_2)
- net GND: now also J10.3 (Pin_3), J4.3 (Pin_3), J5.3 (Pin_3), J9.3 (Pin_3), U13.11 (V-), U15.11 (V-)
- net V1: now also U13.3 (+)
- net V2: now also U13.5 (+)
- net V3: now also U13.10 (+)
- net V4: now also U13.12 (+)
- net at R17.2, R23.2: now also U15.10 (+)
- net at R26.2, U2.3 (CH2): now also U15.8
- net at R20.2, R26.1: now also U15.9 (-)
- net at R16.1, R18.1: now also U13.6 (-), U13.7
- net at R16.2, R22.2: now also U15.5 (+)
- net at R24.2, U2.1 (CH0): now also U15.1
- net at R18.2, R24.1: now also U15.2 (-)
- net at R15.2, R21.2: now also U15.3 (+)
- net at R15.1: now also U13.1, U13.2 (-)
- net at R19.2, R25.1: now also U15.6 (-)
- net at R25.2, U2.2 (CH1): now also U15.7
- net at R17.1, R19.1: now also U13.8, U13.9 (-)
- net at R20.1, U2.4 (CH3): now also U13.13 (-), U13.14
- net at U2.5 (CH4): now also J10.1 (Pin_1)
- net at U2.6 (CH5): now also J9.1 (Pin_1)
- net at U2.7 (CH6): now also J4.1 (Pin_1)
- net at U2.8 (CH7): now also J5.1 (Pin_1)
Other:
- note added: "Old Ballast Pot"
- note removed: "Servo Data [5-7]"
