File: BMS.kicad_sch (KiCad schematic)
At the start: 29 parts, among them IC1 BQ7790400PWR, J1 Conn_01x02_Pin, J2 B5B-XH-A, Q1 CSD18534Q5A, Q2 CSD18534Q5A

Commit message: Pushing updated schematics
Parts:
- added F1: 10A, symbol Device:Fuse
- added JP1: Jumper_2_Open, symbol Jumper:Jumper_2_Open
- IC1: value BQ7790400PWR -> BQ7790512PWR
- J1: footprint (none) -> Connector_Phoenix_GMSTB:PhoenixContact_GMSTBA_2,5_7-G_1x07_P7.50mm_Horizontal
- R1, R14, R2, R3, R4, R5, R7, R8, R9: footprint LED_SMD:LED_0805_2012Metric_Pad1.15x1.40mm_HandSolder -> Resistor_SMD:R_0805_2012Metric_Pad1.20x1.40mm_HandSolder
- R10: value 5.1k -> 4.7k; footprint LED_SMD:LED_0805_2012Metric_Pad1.15x1.40mm_HandSolder -> Resistor_SMD:R_0805_2012Metric_Pad1.20x1.40mm_HandSolder
- R11, R13: value 10M -> 1M; footprint LED_SMD:LED_0805_2012Metric_Pad1.15x1.40mm_HandSolder -> Resistor_SMD:R_0805_2012Metric_Pad1.20x1.40mm_HandSolder
- R12: value 5.1k -> 1k; footprint LED_SMD:LED_0805_2012Metric_Pad1.15x1.40mm_HandSolder -> Resistor_SMD:R_0805_2012Metric_Pad1.20x1.40mm_HandSolder
- R6: value WSHP28184L000FEA -> WSHP28185L000FEA; footprint WSHP28184L000FEA -> WSHP28184L000FEA:WSHP28184L000FEA
- TH1: footprint (none) -> Resistor_SMD:R_0805_2012Metric_Pad1.20x1.40mm_HandSolder
Connections:
- net +15V: now also F1.2; no longer J1.1 (Pin_1)
- net GND: now also JP1.2 (B)
- net GNDREF: now also JP1.1 (A)
- new net: F1.1, J1.1 (Pin_1)
Other:
- note added: "BMS Bypass"
- note added: "BMS GND"
- note added: "Main Electronics GND"
- note added: "Main Power Output"
